File: custom_pcb/custom_pcb.sch (KiCad schematic (older format))
At the start: 297 parts, among them J1 USB_mini_micro_B, K0 KEYSW, K1 KEYSW, K10 KEYSW, K11 KEYSW, K12 KEYSW, K13 KEYSW, K14 KEYSW, K15 KEYSW, K16 KEYSW, K17 KEYSW, K18 KEYSW, K19 KEYSW, K2 KEYSW, K20 KEYSW, K21 KEYSW, K22 KEYSW, K23 KEYSW, K24 KEYSW, K25 KEYSW, K26 KEYSW, K27 KEYSW, K28 KEYSW, K29 KEYSW, K3 KEYSW, K30 KEYSW, K31 KEYSW, K32 KEYSW, K33 KEYSW, K34 KEYSW, K35 KEYSW, K36 KEYSW, K37 KEYSW, K38 KEYSW, K39 KEYSW, K4 KEYSW, K40 KEYSW, K41 KEYSW, K42 KEYSW, K43 KEYSW, K44 KEYSW, K45 KEYSW, K46 KEYSW, K47 KEYSW, K48 KEYSW, K49 KEYSW, K5 KEYSW, K50 KEYSW, K51 KEYSW, K52 KEYSW, K53 KEYSW, K54 KEYSW, K55 KEYSW, K56 KEYSW, K57 KEYSW, K58 KEYSW, K59 KEYSW, K6 KEYSW, K60 KEYSW, K61 KEYSW, K62 KEYSW, K63 KEYSW, K64 KEYSW, K65 KEYSW, K66 KEYSW, K67 KEYSW, K68 KEYSW, K69 KEYSW, K7 KEYSW, K70 KEYSW, K71 KEYSW, K72 KEYSW, K73 KEYSW, K74 KEYSW, K75 KEYSW, K76 KEYSW, K77 KEYSW, K78 KEYSW, K79 KEYSW, K8 KEYSW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

Commit message: cpcb major improvements to trackpoint routing
Parts:
- removed SMD_LED0, SMD_LED1, SMD_LED14, SMD_LED2, SMD_LED29, SMD_LED3, SMD_LED4, SMD_LED44, SMD_LED5, SMD_LED59, SMD_LED6, SMD_LED73, SMD_LED74: SMLVN6RGB, cherry_rgb:SMLVN6RGB, symbol SMLVN6RGB
Changed lines of the file:
@@
 Text GLabel 1050 2550 0    60   Input ~ 0
 c14
-Text GLabel 1050 1850 0    60   Input ~ 0
+Text GLabel 3350 3250 0    60   Input ~ 0
 LED_CLK
 Text GLabel 1050 3250 0    60   Input ~ 0
@@
 Text GLabel 1050 1250 0    60   Input ~ 0
 LED_DATA2
-Text GLabel 1050 3950 0    60   Input ~ 0
+Text GLabel 1050 3650 0    60   Input ~ 0
 TP_DATA
-Text GLabel 1050 3450 0    60   Input ~ 0
+Text GLabel 3350 3150 0    60   Input ~ 0
 TP_CLK
 Text GLabel 4500 2500 1    60   Input ~ 0
 GND
-Text GLabel 4400 2500 1    60   Input ~ 0
+Text GLabel 4200 2500 1    60   Input ~ 0
 TP_DATA
 Text GLabel 4300 2500 1    60   Input ~ 0
 TP_CLK
-Text GLabel 4200 2500 1    60   Input ~ 0
-TP_RST
 Text GLabel 4100 2500 1    60   Input ~ 0
+TP_RST
+Text GLabel 4400 2500 1    60   Input ~ 0
 TP_5V
 Text GLabel 3800 2500 1    60   Input ~ 0
@@
 	1    0    0    -1
 $EndComp
-$Comp
-L SMLVN6RGB SMD_LED73
-U 1 1 58B5FB24
-P 14900 5400
-F 0 "SMD_LED73" H 14900 5770 50  0000 C CNN
-F 1 "SMLVN6RGB" H 14900 5050 50  0000 C CNN
-F 2 "cherry_rgb:SMLVN6RGB" H 14900 5350 50  0001 C CNN
-F 3 "" H 14900 5350 50  0000 C CNN
-	1    14900 5400
-	1    0    0    -1
-$EndComp
-$Comp
-L SMLVN6RGB SMD_LED74
-U 1 1 58B5FB2A
-P 15400 5400
-F 0 "SMD_LED74" H 15400 5770 50  0000 C CNN
-F 1 "SMLVN6RGB" H 15400 5050 50  0000 C CNN
-F 2 "cherry_rgb:SMLVN6RGB" H 15400 5350 50  0001 C CNN
-F 3 "" H 15400 5350 50  0000 C CNN
-	1    15400 5400
-	1    0    0    -1
-$EndComp
 Connection ~ 15100 5150
 Wire Wire Line
@@
 	1    0    0    -1
 $EndComp
-$Comp
-L SMLVN6RGB SMD_LED59
-U 1 1 58B5FC17
-P 15400 4550
-F 0 "SMD_LED59" H 15400 4920 50  0000 C CNN
-F 1 "SMLVN6RGB" H 15400 4200 50  0000 C CNN
-F 2 "cherry_rgb:SMLVN6RGB" H 15400 4500 50  0001 C CNN
-F 3 "" H 15400 4500 50  0000 C CNN
-	1    15400 4550
-	1    0    0    -1
-$EndComp
 Connection ~ 15100 4300
 Wire Wire Line
@@
 	1    0    0    -1
 $EndComp
-$Comp
-L SMLVN6RGB SMD_LED44
-U 1 1 58B5FD04
-P 15400 3700
-F 0 "SMD_LED44" H 15400 4070 50  0000 C CNN
-F 1 "SMLVN6RGB" H 15400 3350 50  0000 C CNN
-F 2 "cherry_rgb:SMLVN6RGB" H 15400 3650 50  0001 C CNN
-F 3 "" H 15400 3650 50  0000 C CNN
-	1    15400 3700
-	1    0    0    -1
-$EndComp
 Connection ~ 15100 3450
 Wire Wire Line
@@
 	1    0    0    -1
 $EndComp
-$Comp
-L SMLVN6RGB SMD_LED29
-U 1 1 58B5FDF1
-P 15400 2850
-F 0 "SMD_LED29" H 15400 3220 50  0000 C CNN
-F 1 "SMLVN6RGB" H 15400 2500 50  0000 C CNN
-F 2 "cherry_rgb:SMLVN6RGB" H 15400 2800 50  0001 C CNN
-F 3 "" H 15400 2800 50  0000 C CNN
-	1    15400 2850
-	1    0    0    -1
-$EndComp
 Connection ~ 15100 2600
 Wire Wire Line
@@
 Connection ~ 8200 3050
 $Comp
-L SMLVN6RGB SMD_LED0
-U 1 1 58B5FE8A
-P 8400 2000
-F 0 "SMD_LED0" H 8400 2370 50  0000 C CNN
-F 1 "SMLVN6RGB" H 8400 1650 50  0000 C CNN
-F 2 "cherry_rgb:SMLVN6RGB" H 8400 1950 50  0001 C CNN
-F 3 "" H 8400 1950 50  0000 C CNN
-	1    8400 2000
-	1    0    0    -1
-$EndComp
-$Comp
-L SMLVN6RGB SMD_LED1
-U 1 1 58B5FE90
-P 8900 2000
-F 0 "SMD_LED1" H 8900 2370 50  0000 C CNN
-F 1 "SMLVN6RGB" H 8900 1650 50  0000 C CNN
-F 2 "cherry_rgb:SMLVN6RGB" H 8900 1950 50  0001 C CNN
-F 3 "" H 8900 1950 50  0000 C CNN
-	1    8900 2000
-	1    0    0    -1
-$EndComp
-$Comp
-L SMLVN6RGB SMD_LED2
-U 1 1 58B5FE96
-P 9400 2000
-F 0 "SMD_LED2" H 9400 2370 50  0000 C CNN
-F 1 "SMLVN6RGB" H 9400 1650 50  0000 C CNN
-F 2 "cherry_rgb:SMLVN6RGB" H 9400 1950 50  0001 C CNN
-F 3 "" H 9400 1950 50  0000 C CNN
-	1    9400 2000
-	1    0    0    -1
-$EndComp
-$Comp
-L SMLVN6RGB SMD_LED3
-U 1 1 58B5FE9C
-P 9900 2000
-F 0 "SMD_LED3" H 9900 2370 50  0000 C CNN
-F 1 "SMLVN6RGB" H 9900 1650 50  0000 C CNN
-F 2 "cherry_rgb:SMLVN6RGB" H 9900 1950 50  0001 C CNN
-F 3 "" H 9900 1950 50  0000 C CNN
-	1    9900 2000
-	1    0    0    -1
-$EndComp
-$Comp
-L SMLVN6RGB SMD_LED4
-U 1 1 58B5FEA2
-P 10400 2000
-F 0 "SMD_LED4" H 10400 2370 50  0000 C CNN
-F 1 "SMLVN6RGB" H 10400 1650 50  0000 C CNN
-F 2 "cherry_rgb:SMLVN6RGB" H 10400 1950 50  0001 C CNN
-F 3 "" H 10400 1950 50  0000 C CNN
-	1    10400 2000
-	1    0    0    -1
-$EndComp
-$Comp
-L SMLVN6RGB SMD_LED5
-U 1 1 58B5FEA8
-P 10900 2000
-F 0 "SMD_LED5" H 10900 2370 50  0000 C CNN
-F 1 "SMLVN6RGB" H 10900 1650 50  0000 C CNN
-F 2 "cherry_rgb:SMLVN6RGB" H 10900 1950 50  0001 C CNN
-F 3 "" H 10900 1950 50  0000 C CNN
-	1    10900 2000
-	1    0    0    -1
-$EndComp
-$Comp
-L SMLVN6RGB SMD_LED6
-U 1 1 58B5FEAE
-P 11400 2000
-F 0 "SMD_LED6" H 11400 2370 50  0000 C CNN
-F 1 "SMLVN6RGB" H 11400 1650 50  0000 C CNN
-F 2 "cherry_rgb:SMLVN6RGB" H 11400 1950 50  0001 C CNN
-F 3 "" H 11400 1950 50  0000 C CNN
-	1    11400 2000
-	1    0    0    -1
-$EndComp
-$Comp
 L SMLVN6RGB SMD_LED7
 U 1 1 58B5FEB4
@@
 	1    0    0    -1
 $EndComp
-$Comp
-L SMLVN6RGB SMD_LED14
-U 1 1 58B5FEDE
-P 15400 2000
-F 0 "SMD_LED14" H 15400 2370 50  0000 C CNN
-F 1 "SMLVN6RGB" H 15400 1650 50  0000 C CNN
-F 2 "cherry_rgb:SMLVN6RGB" H 15400 1950 50  0001 C CNN
-F 3 "" H 15400 1950 50  0000 C CNN
-	1    15400 2000
-	1    0    0    -1
-$EndComp
 Connection ~ 15100 1750
 Wire Wire Line
@@
 Text GLabel 11500 9800 2    60   Input ~ 0
 red0
+Text GLabel 1050 3550 0    60   Input ~ 0
+TP_RST
 $EndSCHEMATC

Commit message: finished 2nd draft led wiring
Changed lines of the file:
@@
 Text GLabel 1050 2550 0    60   Input ~ 0
 c14
-Text GLabel 3350 3250 0    60   Input ~ 0
+Text GLabel 1050 4150 0    60   Input ~ 0
 LED_CLK
 Text GLabel 1050 3250 0    60   Input ~ 0
@@
 Text GLabel 1050 3650 0    60   Input ~ 0
 TP_DATA
-Text GLabel 3350 3150 0    60   Input ~ 0
+Text GLabel 1050 1850 0    60   Input ~ 0
 TP_CLK
 Text GLabel 4500 2500 1    60   Input ~ 0
