File: custom_pcb/custom_pcb.sch (KiCad schematic (older format))
At the start: 293 parts, among them J1 USB_mini_micro_B, K0 KEYSW, K1 KEYSW, K10 KEYSW, K11 KEYSW, K12 KEYSW, K13 KEYSW, K14 KEYSW, K15 KEYSW, K16 KEYSW, K17 KEYSW, K18 KEYSW, K19 KEYSW, K2 KEYSW, K20 KEYSW, K21 KEYSW, K22 KEYSW, K23 KEYSW, K24 KEYSW, K25 KEYSW, K26 KEYSW, K27 KEYSW, K28 KEYSW, K29 KEYSW, K3 KEYSW, K30 KEYSW, K31 KEYSW, K32 KEYSW, K33 KEYSW, K34 KEYSW, K35 KEYSW, K36 KEYSW, K37 KEYSW, K38 KEYSW, K39 KEYSW, K4 KEYSW, K40 KEYSW, K41 KEYSW, K42 KEYSW, K43 KEYSW, K44 KEYSW, K45 KEYSW, K46 KEYSW, K47 KEYSW, K48 KEYSW, K49 KEYSW, K5 KEYSW, K50 KEYSW, K51 KEYSW, K52 KEYSW, K53 KEYSW, K54 KEYSW, K55 KEYSW, K56 KEYSW, K57 KEYSW, K58 KEYSW, K59 KEYSW, K6 KEYSW, K60 KEYSW, K61 KEYSW, K62 KEYSW, K63 KEYSW, K64 KEYSW, K65 KEYSW, K66 KEYSW, K67 KEYSW, K68 KEYSW, K69 KEYSW, K7 KEYSW, K70 KEYSW, K71 KEYSW, K72 KEYSW, K73 KEYSW, K74 KEYSW, K75 KEYSW, K76 KEYSW, K77 KEYSW, K78 KEYSW, K79 KEYSW, K8 KEYSW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

Commit message: cpcb starting to rework led positioning to minimize wiring
Parts:
- removed D60, D61, D62: D, Diodes_SMD:D_SOD-123, symbol D
- removed K60, K61, K62: KEYSW, cherry_rgb:CHERRY_PLATE_NH_100H, symbol KEYSW
Connections:
- net labels added: LED_LE, LED_OE
- net labels removed: r6
- wire segments 2488 -> 4099
Other:
- moved on the sheet: D55, D56, D57, D58, D59, D63, D65, D66, D68, D69, D70, D72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

Commit message: cpcb transistors
Parts:
- removed SLD13: SMLVN6RGB_CA, cherry_rgb:SMLVN6RGB_CA, symbol SMLVN6RGB_CA
- added Q0, Q1, Q2, Q3: Si3993CDV, TO_SOT_Packages_SMD:SOT-23-6_Handsoldering, symbol Si3993CDV
- K1, K2, K3, K4, K5, K6, K63, K67, K68, K7, K8, K9: footprint cherry_rgb:CHERRY_PLATE_NH_100H -> cherry_rgb:CHERRY_PLATE_91.6H
Connections:
- net labels added: +3.3V, as0, as1, as2, as3, as4, as5, as6
- net labels removed: V3.3
- wire segments 4099 -> 2491
