File: custom_pcb/custom_pcb.kicad_pcb (KiCad board)
At the start: 2 copper layers, 285 x 152 mm, 312 parts, among them J1 USB_mini_micro_B, K0 KEYSW, K1 KEYSW, K10 KEYSW, K11 KEYSW, K12 KEYSW, K13 KEYSW, K14 KEYSW, K15 KEYSW, K16 KEYSW, K17 KEYSW, K18 KEYSW, K19 KEYSW, K2 KEYSW, K20 KEYSW, K21 KEYSW, K22 KEYSW, K23 KEYSW, K24 KEYSW, K25 KEYSW, K26 KEYSW, K27 KEYSW, K28 KEYSW, K29 KEYSW, K3 KEYSW, K30 KEYSW, K31 KEYSW, K32 KEYSW, K33 KEYSW, K34 KEYSW, K35 KEYSW, K36 KEYSW, K37 KEYSW, K38 KEYSW, K39 KEYSW, K4 KEYSW, K40 KEYSW, K41 KEYSW, K42 KEYSW, K43 KEYSW, K44 KEYSW, K45 KEYSW, K46 KEYSW, K47 KEYSW, K48 KEYSW, K49 KEYSW, K5 KEYSW, K50 KEYSW, K51 KEYSW, K52 KEYSW, K53 KEYSW, K54 KEYSW, K55 KEYSW, K56 KEYSW, K57 KEYSW, K58 KEYSW, K59 KEYSW, K60 KEYSW, K63 KEYSW, K64 KEYSW, K65 KEYSW, K66 KEYSW, K67 KEYSW, K68 KEYSW, K69 KEYSW, K7 KEYSW, K70 KEYSW, K71 KEYSW, K72 KEYSW, K73 KEYSW, K74 KEYSW, K75 KEYSW, K76 KEYSW, K77 KEYSW, K78 KEYSW, K79 KEYSW, K8 KEYSW, K80 KEYSW, K81 KEYSW, K82 KEYSW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

Commit message: about to try an alternate rout
Routing:
- net Net-(LC2-Pad23): track 30.1 -> 31.3 mm
Changed lines of the file:
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@@
     (thickness 1.6)
     (drawings 6)
-    (tracks 1898)
+    (tracks 1901)
     (zones 0)
     (modules 312)
@@
   (segment (start 138.325 59.575) (end 143 64.25) (width 0.25) (layer B.Cu) (net 165))
   (segment (start 138.325 51.6) (end 138.325 59.575) (width 0.25) (layer B.Cu) (net 165))
-  (segment (start 155.75 53.635002) (end 159.895984 53.635002) (width 0.25) (layer F.Cu) (net 166))
+  (segment (start 151.25 42.5) (end 152 43.25) (width 0.25) (layer F.Cu) (net 166))
+  (segment (start 152.25 43.25) (end 152.75 43.75) (width 0.25) (layer F.Cu) (net 166))
+  (segment (start 152 43.25) (end 152.25 43.25) (width 0.25) (layer F.Cu) (net 166))
+  (segment (start 152.75 43.75) (end 152.75 44.25) (width 0.25) (layer F.Cu) (net 166))
+  (segment (start 152.75 44.25) (end 152.5 44.5) (width 0.25) (layer F.Cu) (net 166))
+  (segment (start 152.5 44.5) (end 152.5 48) (width 0.25) (layer F.Cu) (net 166))
+  (segment (start 152 48.5) (end 152 51) (width 0.25) (layer F.Cu) (net 166))
+  (segment (start 152 51) (end 154.635002 53.635002) (width 0.25) (layer F.Cu) (net 166))
+  (segment (start 154.635002 53.635002) (end 159.895984 53.635002) (width 0.25) (layer F.Cu) (net 166))
   (segment (start 159.895984 53.635002) (end 165 58.739018) (width 0.25) (layer F.Cu) (net 166))
+  (segment (start 152.5 48) (end 152 48.5) (width 0.25) (layer F.Cu) (net 166))
   (segment (start 150.75 42.5) (end 151.25 42.5) (width 0.25) (layer B.Cu) (net 166))
   (segment (start 149 42.75) (end 150.5 42.75) (width 0.25) (layer B.Cu) (net 166))
@@
   (segment (start 150.5 42.75) (end 150.75 42.5) (width 0.25) (layer B.Cu) (net 166))
   (segment (start 149.325 45.6) (end 149.325 44.8) (width 0.25) (layer B.Cu) (net 166))
-  (segment (start 151.25 42.5) (end 152 43.25) (width 0.25) (layer F.Cu) (net 166))
-  (segment (start 152 43.25) (end 152.25 43.25) (width 0.25) (layer F.Cu) (net 166))
-  (segment (start 152.25 43.25) (end 152.75 43.75) (width 0.25) (layer F.Cu) (net 166))
-  (segment (start 152.75 50.635002) (end 153 50.885002) (width 0.25) (layer F.Cu) (net 166))
-  (segment (start 153 50.885002) (end 155.75 53.635002) (width 0.25) (layer F.Cu) (net 166))
-  (segment (start 152.75 43.75) (end 152.75 50.635002) (width 0.25) (layer F.Cu) (net 166))
   (via (at 151.25 42.5) (size 0.6) (drill 0.4) (layers F.Cu B.Cu) (net 166))
   (segment (start 88.2 31.75) (end 88.2 32.7) (width 0.25) (layer B.Cu) (net 167))
