File: test_pcb/_saved_test_pcb.sch (KiCad schematic (older format))
At the start: 76 parts, among them K0 KEYSW, K1 KEYSW, K10 KEYSW, K12 KEYSW, K13 KEYSW, K14 KEYSW, K15 KEYSW, K16 KEYSW, K17 KEYSW, K18 KEYSW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

Commit message: test groundplanes
Parts:
- added P10, P11, P12, P13, P14, P15, P4, P5, P6, P7, P8, P9: CONN_01X01, cherry_rgb:VIA127, symbol CONN_01X01
