File: test_pcb/test_pcb.sch (KiCad schematic (older format))
At the start: 71 parts, among them K0 KEYSW, K1 KEYSW, K10 KEYSW, K12 KEYSW, K13 KEYSW, K14 KEYSW, K15 KEYSW, K16 KEYSW, K17 KEYSW, K18 KEYSW, K2 KEYSW, K20 KEYSW, K21 KEYSW, K22 KEYSW, K3 KEYSW, K4 KEYSW, K5 KEYSW, K6 KEYSW, K7 KEYSW, K8 KEYSW, K9 KEYSW, P0 CONN_01X08, P1 CONN_01X08, P2 CONN_01X08, U0 Teensy3.2, U1 STP16CP05

Commit message: test output holes
Parts:
- P1, P2: footprint Connectors_Molex:Molex_PicoBlade_53261-0871_08x1.25mm_Angled -> Socket_Strips:Socket_Strip_Straight_1x08_Pitch2.54mm
- R0: footprint (none) -> Resistors_SMD:R_0603_HandSoldering
- R1, R2: renamed from R?; footprint (none) -> Resistors_SMD:R_0603_HandSoldering
Changed lines of the file:
@@
 F 0 "R0" V 7980 3550 50  0000 C CNN
 F 1 "R" V 7900 3550 50  0000 C CNN
-F 2 "" H 7900 3550 60  0000 C CNN
+F 2 "Resistors_SMD:R_0603_HandSoldering" H 7900 3550 60  0001 C CNN
 F 3 "" H 7900 3550 60  0000 C CNN
 	1    7900 3550
@@
 $EndComp
 $Comp
-L R R?
+L R R1
 U 1 1 58A3D3E0
 P 7900 3650
-F 0 "R?" V 7980 3650 50  0000 C CNN
+F 0 "R1" V 7980 3650 50  0000 C CNN
 F 1 "R" V 7900 3650 50  0000 C CNN
-F 2 "" H 7900 3650 60  0000 C CNN
+F 2 "Resistors_SMD:R_0603_HandSoldering" H 7900 3650 60  0001 C CNN
 F 3 "" H 7900 3650 60  0000 C CNN
 	1    7900 3650
@@
 $EndComp
 $Comp
-L R R?
+L R R2
 U 1 1 58A3D4D0
 P 7900 3750
-F 0 "R?" V 7980 3750 50  0000 C CNN
+F 0 "R2" V 7980 3750 50  0000 C CNN
 F 1 "R" V 7900 3750 50  0000 C CNN
-F 2 "" H 7900 3750 60  0000 C CNN
+F 2 "Resistors_SMD:R_0603_HandSoldering" H 7900 3750 60  0001 C CNN
 F 3 "" H 7900 3750 60  0000 C CNN
 	1    7900 3750
@@
 F 0 "P1" H 7950 5900 50  0000 C CNN
 F 1 "CONN_01X08" V 8050 5450 50  0000 C CNN
-F 2 "Connectors_Molex:Molex_PicoBlade_53261-0871_08x1.25mm_Angled" H 7950 5450 50  0001 C CNN
+F 2 "Socket_Strips:Socket_Strip_Straight_1x08_Pitch2.54mm" H 7950 5450 50  0001 C CNN
 F 3 "" H 7950 5450 50  0000 C CNN
 	1    7950 5450
@@
 F 0 "P2" H 7950 6700 50  0000 C CNN
 F 1 "CONN_01X08" V 8050 6250 50  0000 C CNN
-F 2 "Connectors_Molex:Molex_PicoBlade_53261-0871_08x1.25mm_Angled" H 7950 6250 50  0001 C CNN
+F 2 "Socket_Strips:Socket_Strip_Straight_1x08_Pitch2.54mm" H 7950 6250 50  0001 C CNN
 F 3 "" H 7950 6250 50  0000 C CNN
 	1    7950 6250

Commit message: test pcb freerouting is bugged on this right now
Parts:
- removed P0: CONN_01X08, Connectors_Molex:Molex_PicoBlade_53261-0871_08x1.25mm_Angled, symbol CONN_01X08
- removed U0: Teensy3.2, Teensy:Teensy30_31_32_LC, symbol Teensy3.2
Connections:
- net labels removed: BTN0, BTN1, BTN2, DATA, TP_CLK, TP_RST, VCC
- wire segments 243 -> 242
Other:
- moved on the sheet: P1, P2
Changed lines of the file:
@@
 Comment4 ""
 $EndDescr
-$Comp
-L Teensy3.2 U0
-U 1 1 5894073C
-P 10000 2000
-F 0 "U0" H 10000 3500 60  0000 C CNN
-F 1 "Teensy3.2" H 10000 500 60  0000 C CNN
-F 2 "Teensy:Teensy30_31_32_LC" H 10000 1200 60  0001 C CNN
-F 3 "" H 10000 1200 60  0000 C CNN
-	1    10000 2000
-	1    0    0    -1
-$EndComp
 NoConn ~ -3200 7450
-$Comp
-L CONN_01X08 P0
-U 1 1 5897F60A
-P 9900 5300
-F 0 "P0" H 9900 5750 50  0000 C CNN
-F 1 "CONN_01X08" V 10000 5300 50  0000 C CNN
-F 2 "Connectors_Molex:Molex_PicoBlade_53261-0871_08x1.25mm_Angled" H 9900 5300 50  0001 C CNN
-F 3 "" H 9900 5300 50  0000 C CNN
-	1    9900 5300
-	1    0    0    -1
-$EndComp
-Text GLabel 9700 5650 0    60   Input ~ 0
-BTN0
-Text GLabel 9700 5550 0    60   Input ~ 0
-BTN1
-Text GLabel 9700 5450 0    60   Input ~ 0
-BTN2
-Text GLabel 9700 5350 0    60   Input ~ 0
-VCC
-Text GLabel 9700 5050 0    60   Input ~ 0
-DATA
-Text GLabel 9700 5250 0    60   Input ~ 0
-TP_RST
-Text GLabel 9700 5150 0    60   Input ~ 0
-TP_CLK
 $Comp
 L SMLVN6RGB SMD_LED0
@@
 a3-17-2
 $Comp
-L GND #PWR01
-U 1 1 58A59EDB
-P 9450 4950
-F 0 "#PWR01" H 9450 4700 50  0001 C CNN
-F 1 "GND" H 9450 4800 50  0000 C CNN
-F 2 "" H 9450 4950 50  0000 C CNN
-F 3 "" H 9450 4950 50  0000 C CNN
-	1    9450 4950
-	0    1    1    0
-$EndComp
-Wire Wire Line
-	9700 4950 9450 4950
-$Comp
 L GND #PWR02
 U 1 1 58A5AE89
@@
 	0    1    1    0
 $EndComp
-Text GLabel 7750 5100 0    60   Input ~ 0
+Text GLabel 8000 4800 0    60   Input ~ 0
 a3-10-0
-Text GLabel 7750 5200 0    60   Input ~ 0
+Text GLabel 8000 4900 0    60   Input ~ 0
 a3-10-1
-Text GLabel 7750 5300 0    60   Input ~ 0
+Text GLabel 8000 5000 0    60   Input ~ 0
 a3-10-2
-Text GLabel 7750 5400 0    60   Input ~ 0
+Text GLabel 8000 5100 0    60   Input ~ 0
 a3-17-0
-Text GLabel 7750 5500 0    60   Input ~ 0
+Text GLabel 8000 5200 0    60   Input ~ 0
 a3-17-1
-Text GLabel 7750 5600 0    60   Input ~ 0
+Text GLabel 8000 5300 0    60   Input ~ 0
 a3-17-2
 $Comp
@@
 L CONN_01X08 P1
 U 1 1 58A3B45B
-P 7950 5450
-F 0 "P1" H 7950 5900 50  0000 C CNN
-F 1 "CONN_01X08" V 8050 5450 50  0000 C CNN
-F 2 "Socket_Strips:Socket_Strip_Straight_1x08_Pitch2.54mm" H 7950 5450 50  0001 C CNN
-F 3 "" H 7950 5450 50  0000 C CNN
-	1    7950 5450
+P 8200 5150
+F 0 "P1" H 8200 5600 50  0000 C CNN
+F 1 "CONN_01X08" V 8300 5150 50  0000 C CNN
+F 2 "Socket_Strips:Socket_Strip_Straight_1x08_Pitch2.54mm" H 8200 5150 50  0001 C CNN
+F 3 "" H 8200 5150 50  0000 C CNN
+	1    8200 5150
 	1    0    0    -1
 $EndComp
@@
 L CONN_01X08 P2
 U 1 1 58A3CB40
-P 7950 6250
-F 0 "P2" H 7950 6700 50  0000 C CNN
-F 1 "CONN_01X08" V 8050 6250 50  0000 C CNN
-F 2 "Socket_Strips:Socket_Strip_Straight_1x08_Pitch2.54mm" H 7950 6250 50  0001 C CNN
-F 3 "" H 7950 6250 50  0000 C CNN
-	1    7950 6250
-	1    0    0    -1
-$EndComp
-Text GLabel 7750 5700 0    60   Input ~ 0
+P 7000 6050
+F 0 "P2" H 7000 6500 50  0000 C CNN
+F 1 "CONN_01X08" V 7100 6050 50  0000 C CNN
+F 2 "Socket_Strips:Socket_Strip_Straight_1x08_Pitch2.54mm" H 7000 6050 50  0001 C CNN
+F 3 "" H 7000 6050 50  0000 C CNN
+	1    7000 6050
+	1    0    0    -1
+$EndComp
+Text GLabel 8000 5400 0    60   Input ~ 0
 blue1
-Text GLabel 7750 5800 0    60   Input ~ 0
+Text GLabel 8000 5500 0    60   Input ~ 0
 red1
-Text GLabel 7750 5900 0    60   Input ~ 0
+Text GLabel 6800 5700 0    60   Input ~ 0
 green1
-Text GLabel 7750 6000 0    60   Input ~ 0
+Text GLabel 6800 5800 0    60   Input ~ 0
 blue2
-Text GLabel 7750 6100 0    60   Input ~ 0
+Text GLabel 6800 5900 0    60   Input ~ 0
 red2
-Text GLabel 7800 6200 0    60   Input ~ 0
+Text GLabel 6850 6000 0    60   Input ~ 0
 green2
 $EndSCHEMATC

Commit message: test pcb some improvement, but still getting the infinite fails
Parts:
- added P3: CONN_01X06, Socket_Strips:Socket_Strip_Straight_1x06_Pitch2.54mm, symbol CONN_01X06
- SMD_LED0, SMD_LED1, SMD_LED11, SMD_LED12, SMD_LED13, SMD_LED14, SMD_LED15, SMD_LED16, SMD_LED18, SMD_LED19, SMD_LED2, SMD_LED20, SMD_LED3, SMD_LED4, SMD_LED5, SMD_LED6, SMD_LED7, SMD_LED8, SMD_LED9: value SMLVN6RGB -> SMLVN6RGB_CA; footprint cherry_rgb:SMLVN6RGB -> cherry_rgb:SMLVN6RGB_CA; symbol SMLVN6RGB -> SMLVN6RGB_CA
Changed lines of the file:
@@
 NoConn ~ -3200 7450
 $Comp
-L SMLVN6RGB SMD_LED0
+L SMLVN6RGB_CA SMD_LED0
 U 1 1 58A0BD18
 P 1000 1000
 F 0 "SMD_LED0" H 1000 1370 50  0000 C CNN
-F 1 "SMLVN6RGB" H 1000 650 50  0000 C CNN
-F 2 "cherry_rgb:SMLVN6RGB" H 1000 950 50  0001 C CNN
+F 1 "SMLVN6RGB_CA" H 1000 650 50  0000 C CNN
+F 2 "cherry_rgb:SMLVN6RGB_CA" H 1000 950 50  0001 C CNN
 F 3 "" H 1000 950 50  0000 C CNN
 	1    1000 1000
@@
 $EndComp
 $Comp
-L SMLVN6RGB SMD_LED1
+L SMLVN6RGB_CA SMD_LED1
 U 1 1 58A0BED8
 P 1700 1000
 F 0 "SMD_LED1" H 1700 1370 50  0000 C CNN
-F 1 "SMLVN6RGB" H 1700 650 50  0000 C CNN
-F 2 "cherry_rgb:SMLVN6RGB" H 1700 950 50  0001 C CNN
+F 1 "SMLVN6RGB_CA" H 1700 650 50  0000 C CNN
+F 2 "cherry_rgb:SMLVN6RGB_CA" H 1700 950 50  0001 C CNN
 F 3 "" H 1700 950 50  0000 C CNN
 	1    1700 1000
@@
 $EndComp
 $Comp
-L SMLVN6RGB SMD_LED2
+L SMLVN6RGB_CA SMD_LED2
 U 1 1 58A0BF71
 P 2400 1000
 F 0 "SMD_LED2" H 2400 1370 50  0000 C CNN
-F 1 "SMLVN6RGB" H 2400 650 50  0000 C CNN
-F 2 "cherry_rgb:SMLVN6RGB" H 2400 950 50  0001 C CNN
+F 1 "SMLVN6RGB_CA" H 2400 650 50  0000 C CNN
+F 2 "cherry_rgb:SMLVN6RGB_CA" H 2400 950 50  0001 C CNN
 F 3 "" H 2400 950 50  0000 C CNN
 	1    2400 1000
@@
 $EndComp
 $Comp
-L SMLVN6RGB SMD_LED3
+L SMLVN6RGB_CA SMD_LED3
 U 1 1 58A0C01B
 P 3100 1000
 F 0 "SMD_LED3" H 3100 1370 50  0000 C CNN
-F 1 "SMLVN6RGB" H 3100 650 50  0000 C CNN
-F 2 "cherry_rgb:SMLVN6RGB" H 3100 950 50  0001 C CNN
+F 1 "SMLVN6RGB_CA" H 3100 650 50  0000 C CNN
+F 2 "cherry_rgb:SMLVN6RGB_CA" H 3100 950 50  0001 C CNN
 F 3 "" H 3100 950 50  0000 C CNN
 	1    3100 1000
@@
 $EndComp
 $Comp
-L SMLVN6RGB SMD_LED4
+L SMLVN6RGB_CA SMD_LED4
 U 1 1 58A0E407
 P 3800 1000
 F 0 "SMD_LED4" H 3800 1370 50  0000 C CNN
-F 1 "SMLVN6RGB" H 3800 650 50  0000 C CNN
-F 2 "cherry_rgb:SMLVN6RGB" H 3800 950 50  0001 C CNN
+F 1 "SMLVN6RGB_CA" H 3800 650 50  0000 C CNN
+F 2 "cherry_rgb:SMLVN6RGB_CA" H 3800 950 50  0001 C CNN
 F 3 "" H 3800 950 50  0000 C CNN
 	1    3800 1000
@@
 $EndComp
 $Comp
-L SMLVN6RGB SMD_LED5
+L SMLVN6RGB_CA SMD_LED5
 U 1 1 58A0E40D
 P 4500 1000
 F 0 "SMD_LED5" H 4500 1370 50  0000 C CNN
-F 1 "SMLVN6RGB" H 4500 650 50  0000 C CNN
-F 2 "cherry_rgb:SMLVN6RGB" H 4500 950 50  0001 C CNN
+F 1 "SMLVN6RGB_CA" H 4500 650 50  0000 C CNN
+F 2 "cherry_rgb:SMLVN6RGB_CA" H 4500 950 50  0001 C CNN
 F 3 "" H 4500 950 50  0000 C CNN
 	1    4500 1000
@@
 $EndComp
 $Comp
-L SMLVN6RGB SMD_LED6
+L SMLVN6RGB_CA SMD_LED6
 U 1 1 58A0E413
 P 5200 1000
 F 0 "SMD_LED6" H 5200 1370 50  0000 C CNN
-F 1 "SMLVN6RGB" H 5200 650 50  0000 C CNN
-F 2 "cherry_rgb:SMLVN6RGB" H 5200 950 50  0001 C CNN
+F 1 "SMLVN6RGB_CA" H 5200 650 50  0000 C CNN
+F 2 "cherry_rgb:SMLVN6RGB_CA" H 5200 950 50  0001 C CNN
 F 3 "" H 5200 950 50  0000 C CNN
 	1    5200 1000
@@
 $EndComp
 $Comp
-L SMLVN6RGB SMD_LED7
+L SMLVN6RGB_CA SMD_LED7
 U 1 1 58A100CF
 P 1000 1850
 F 0 "SMD_LED7" H 1000 2220 50  0000 C CNN
-F 1 "SMLVN6RGB" H 1000 1500 50  0000 C CNN
-F 2 "cherry_rgb:SMLVN6RGB" H 1000 1800 50  0001 C CNN
+F 1 "SMLVN6RGB_CA" H 1000 1500 50  0000 C CNN
+F 2 "cherry_rgb:SMLVN6RGB_CA" H 1000 1800 50  0001 C CNN
 F 3 "" H 1000 1800 50  0000 C CNN
 	1    1000 1850
@@
 $EndComp
 $Comp
-L SMLVN6RGB SMD_LED8
+L SMLVN6RGB_CA SMD_LED8
 U 1 1 58A100D5
 P 1700 1850
 F 0 "SMD_LED8" H 1700 2220 50  0000 C CNN
-F 1 "SMLVN6RGB" H 1700 1500 50  0000 C CNN
-F 2 "cherry_rgb:SMLVN6RGB" H 1700 1800 50  0001 C CNN
+F 1 "SMLVN6RGB_CA" H 1700 1500 50  0000 C CNN
+F 2 "cherry_rgb:SMLVN6RGB_CA" H 1700 1800 50  0001 C CNN
 F 3 "" H 1700 1800 50  0000 C CNN
 	1    1700 1850
@@
 $EndComp
 $Comp
-L SMLVN6RGB SMD_LED9
+L SMLVN6RGB_CA SMD_LED9
 U 1 1 58A100DB
 P 2400 1850
 F 0 "SMD_LED9" H 2400 2220 50  0000 C CNN
-F 1 "SMLVN6RGB" H 2400 1500 50  0000 C CNN
-F 2 "cherry_rgb:SMLVN6RGB" H 2400 1800 50  0001 C CNN
+F 1 "SMLVN6RGB_CA" H 2400 1500 50  0000 C CNN
+F 2 "cherry_rgb:SMLVN6RGB_CA" H 2400 1800 50  0001 C CNN
 F 3 "" H 2400 1800 50  0000 C CNN
 	1    2400 1850
@@
 $EndComp
 $Comp
-L SMLVN6RGB SMD_LED11
+L SMLVN6RGB_CA SMD_LED11
 U 1 1 58A100E7
 P 3800 1850
 F 0 "SMD_LED11" H 3800 2220 50  0000 C CNN
-F 1 "SMLVN6RGB" H 3800 1500 50  0000 C CNN
-F 2 "cherry_rgb:SMLVN6RGB" H 3800 1800 50  0001 C CNN
+F 1 "SMLVN6RGB_CA" H 3800 1500 50  0000 C CNN
+F 2 "cherry_rgb:SMLVN6RGB_CA" H 3800 1800 50  0001 C CNN
 F 3 "" H 3800 1800 50  0000 C CNN
 	1    3800 1850
@@
 $EndComp
 $Comp
-L SMLVN6RGB SMD_LED12
+L SMLVN6RGB_CA SMD_LED12
 U 1 1 58A100ED
 P 4500 1850
 F 0 "SMD_LED12" H 4500 2220 50  0000 C CNN
-F 1 "SMLVN6RGB" H 4500 1500 50  0000 C CNN
-F 2 "cherry_rgb:SMLVN6RGB" H 4500 1800 50  0001 C CNN
+F 1 "SMLVN6RGB_CA" H 4500 1500 50  0000 C CNN
+F 2 "cherry_rgb:SMLVN6RGB_CA" H 4500 1800 50  0001 C CNN
 F 3 "" H 4500 1800 50  0000 C CNN
 	1    4500 1850
@@
 $EndComp
 $Comp
-L SMLVN6RGB SMD_LED13
+L SMLVN6RGB_CA SMD_LED13
 U 1 1 58A100F3
 P 5200 1850
 F 0 "SMD_LED13" H 5200 2220 50  0000 C CNN
-F 1 "SMLVN6RGB" H 5200 1500 50  0000 C CNN
-F 2 "cherry_rgb:SMLVN6RGB" H 5200 1800 50  0001 C CNN
+F 1 "SMLVN6RGB_CA" H 5200 1500 50  0000 C CNN
+F 2 "cherry_rgb:SMLVN6RGB_CA" H 5200 1800 50  0001 C CNN
 F 3 "" H 5200 1800 50  0000 C CNN
 	1    5200 1850
@@
 $EndComp
 $Comp
-L SMLVN6RGB SMD_LED14
+L SMLVN6RGB_CA SMD_LED14
 U 1 1 58A1042B
 P 1000 2700
 F 0 "SMD_LED14" H 1000 3070 50  0000 C CNN
-F 1 "SMLVN6RGB" H 1000 2350 50  0000 C CNN
-F 2 "cherry_rgb:SMLVN6RGB" H 1000 2650 50  0001 C CNN
+F 1 "SMLVN6RGB_CA" H 1000 2350 50  0000 C CNN
+F 2 "cherry_rgb:SMLVN6RGB_CA" H 1000 2650 50  0001 C CNN
 F 3 "" H 1000 2650 50  0000 C CNN
 	1    1000 2700
@@
 $EndComp
 $Comp
-L SMLVN6RGB SMD_LED15
+L SMLVN6RGB_CA SMD_LED15
 U 1 1 58A10431
 P 1700 2700
 F 0 "SMD_LED15" H 1700 3070 50  0000 C CNN
-F 1 "SMLVN6RGB" H 1700 2350 50  0000 C CNN
-F 2 "cherry_rgb:SMLVN6RGB" H 1700 2650 50  0001 C CNN
+F 1 "SMLVN6RGB_CA" H 1700 2350 50  0000 C CNN
+F 2 "cherry_rgb:SMLVN6RGB_CA" H 1700 2650 50  0001 C CNN
 F 3 "" H 1700 2650 50  0000 C CNN
 	1    1700 2700
@@
 $EndComp
 $Comp
-L SMLVN6RGB SMD_LED16
+L SMLVN6RGB_CA SMD_LED16
 U 1 1 58A10437
 P 2400 2700
 F 0 "SMD_LED16" H 2400 3070 50  0000 C CNN
-F 1 "SMLVN6RGB" H 2400 2350 50  0000 C CNN
-F 2 "cherry_rgb:SMLVN6RGB" H 2400 2650 50  0001 C CNN
+F 1 "SMLVN6RGB_CA" H 2400 2350 50  0000 C CNN
+F 2 "cherry_rgb:SMLVN6RGB_CA" H 2400 2650 50  0001 C CNN
 F 3 "" H 2400 2650 50  0000 C CNN
 	1    2400 2700
@@
 $EndComp
 $Comp
-L SMLVN6RGB SMD_LED18
+L SMLVN6RGB_CA SMD_LED18
 U 1 1 58A10443
 P 3800 2700
 F 0 "SMD_LED18" H 3800 3070 50  0000 C CNN
-F 1 "SMLVN6RGB" H 3800 2350 50  0000 C CNN
-F 2 "cherry_rgb:SMLVN6RGB" H 3800 2650 50  0001 C CNN
+F 1 "SMLVN6RGB_CA" H 3800 2350 50  0000 C CNN
+F 2 "cherry_rgb:SMLVN6RGB_CA" H 3800 2650 50  0001 C CNN
 F 3 "" H 3800 2650 50  0000 C CNN
 	1    3800 2700
@@
 $EndComp
 $Comp
-L SMLVN6RGB SMD_LED19
+L SMLVN6RGB_CA SMD_LED19
 U 1 1 58A10449
 P 4500 2700
 F 0 "SMD_LED19" H 4500 3070 50  0000 C CNN
-F 1 "SMLVN6RGB" H 4500 2350 50  0000 C CNN
-F 2 "cherry_rgb:SMLVN6RGB" H 4500 2650 50  0001 C CNN
+F 1 "SMLVN6RGB_CA" H 4500 2350 50  0000 C CNN
+F 2 "cherry_rgb:SMLVN6RGB_CA" H 4500 2650 50  0001 C CNN
 F 3 "" H 4500 2650 50  0000 C CNN
 	1    4500 2700
@@
 $EndComp
 $Comp
-L SMLVN6RGB SMD_LED20
+L SMLVN6RGB_CA SMD_LED20
 U 1 1 58A1044F
 P 5200 2700
 F 0 "SMD_LED20" H 5200 3070 50  0000 C CNN
-F 1 "SMLVN6RGB" H 5200 2350 50  0000 C CNN
-F 2 "cherry_rgb:SMLVN6RGB" H 5200 2650 50  0001 C CNN
+F 1 "SMLVN6RGB_CA" H 5200 2350 50  0000 C CNN
+F 2 "cherry_rgb:SMLVN6RGB_CA" H 5200 2650 50  0001 C CNN
 F 3 "" H 5200 2650 50  0000 C CNN
 	1    5200 2700
@@
 a3-17-2
 $Comp
-L GND #PWR02
+L GND #PWR01
 U 1 1 58A5AE89
 P 6500 2850
-F 0 "#PWR02" H 6500 2600 50  0001 C CNN
+F 0 "#PWR01" H 6500 2600 50  0001 C CNN
 F 1 "GND" H 6500 2700 50  0000 C CNN
 F 2 "" H 6500 2850 50  0000 C CNN
@@
 a3-17-2
 $Comp
-L +3.3V #PWR03
+L +3.3V #PWR02
 U 1 1 58A3C033
 P 7650 2850
-F 0 "#PWR03" H 7650 2700 50  0001 C CNN
+F 0 "#PWR02" H 7650 2700 50  0001 C CNN
 F 1 "+3.3V" H 7650 2990 50  0000 C CNN
 F 2 "" H 7650 2850 50  0000 C CNN
@@
 Text GLabel 6800 5900 0    60   Input ~ 0
 red2
-Text GLabel 6850 6000 0    60   Input ~ 0
+Text GLabel 6800 6000 0    60   Input ~ 0
 green2
+$Comp
+L CONN_01X06 P3
+U 1 1 58B0E912
+P 5500 5400
+F 0 "P3" H 5500 5750 50  0000 C CNN
+F 1 "CONN_01X06" V 5600 5400 50  0000 C CNN
+F 2 "Socket_Strips:Socket_Strip_Straight_1x06_Pitch2.54mm" H 5500 5400 50  0001 C CNN
+F 3 "" H 5500 5400 50  0000 C CNN
+	1    5500 5400
+	1    0    0    -1
+$EndComp
+Text GLabel 6800 6100 0    60   Input ~ 0
+c0
+Text GLabel 6800 6200 0    60   Input ~ 0
+c1
+Text GLabel 6800 6300 0    60   Input ~ 0
+c2
+Text GLabel 6800 6400 0    60   Input ~ 0
+c3
+Text GLabel 5300 5150 0    60   Input ~ 0
+r0
+Text GLabel 5300 5250 0    60   Input ~ 0
+r1
+Text GLabel 5300 5350 0    60   Input ~ 0
+r2
+Text GLabel 5300 5450 0    60   Input ~ 0
+r3
+Text GLabel 5300 5550 0    60   Input ~ 0
+r4
+Text GLabel 5300 5650 0    60   Input ~ 0
+r5
 $EndSCHEMATC

Commit message: test pcb seem to have fixed the routing bug
Parts:
- added JP1, JP4: Jumper_NC_Small, Pin_Headers:Pin_Header_Angled_1x02_Pitch1.27mm, symbol Jumper_NC_Small
- added JP2, JP3, JP5: Jumper_NC_Dual, Pin_Headers:Pin_Header_Angled_1x03_Pitch1.27mm, symbol Jumper_NC_Dual
- P1: value CONN_01X08 -> CONN_01X10; footprint Socket_Strips:Socket_Strip_Straight_1x08_Pitch2.54mm -> Socket_Strips:Socket_Strip_Straight_1x10_Pitch2.54mm; symbol CONN_01X08 -> CONN_01X10
Connections:
- wire segments 242 -> 254
Other:
- moved on the sheet: R0, R2

Commit message: testp progress
Parts:
- added P10, P11, P12, P13, P14, P15, P4, P5, P6, P7, P8, P9: CONN_01X01, Socket_Strips:Socket_Strip_Straight_1x01_Pitch1.27mm, symbol CONN_01X01
Other:
- moved on the sheet: JP1, JP2, JP3, JP4, JP5, P1, P2, P3, R0, R1, R2, U1

Commit message: test a bit better
Changed lines of the file:
@@
 a3-17-2
 $Comp
-L GND #PWR1
+L GND #PWR01
 U 1 1 58A5AE89
 P 7750 2550
-F 0 "#PWR1" H 7750 2300 50  0001 C CNN
+F 0 "#PWR01" H 7750 2300 50  0001 C CNN
 F 1 "GND" H 7750 2400 50  0000 C CNN
 F 2 "" H 7750 2550 50  0000 C CNN
@@
 a3-17-2
 $Comp
-L +3.3V #PWR2
+L +3.3V #PWR02
 U 1 1 58A3C033
 P 8900 2550
-F 0 "#PWR2" H 8900 2400 50  0001 C CNN
+F 0 "#PWR02" H 8900 2400 50  0001 C CNN
 F 1 "+3.3V" H 8900 2690 50  0000 C CNN
 F 2 "" H 8900 2550 50  0000 C CNN
@@
 Text GLabel 10600 3350 0    60   Input ~ 0
 red1
-Text GLabel 10550 1550 0    60   Input ~ 0
+Text GLabel 10550 1950 0    60   Input ~ 0
 green1
 Text GLabel 10550 4250 0    60   Input ~ 0
@@
 	1    0    0    -1
 $EndComp
+Text GLabel 10550 1350 0    60   Input ~ 0
+c0
+Text GLabel 10550 1450 0    60   Input ~ 0
+c1
+Text GLabel 10550 1550 0    60   Input ~ 0
+c2
 Text GLabel 10550 1650 0    60   Input ~ 0
-c0
-Text GLabel 10550 1750 0    60   Input ~ 0
-c1
-Text GLabel 10550 1850 0    60   Input ~ 0
-c2
-Text GLabel 10550 1950 0    60   Input ~ 0
 c3
 Text GLabel 10550 1250 0    60   Input ~ 0
 r0
-Text GLabel 10550 1350 0    60   Input ~ 0
+Text GLabel 10550 1850 0    60   Input ~ 0
 r1
-Text GLabel 10550 1450 0    60   Input ~ 0
+Text GLabel 10550 1750 0    60   Input ~ 0
 r2
 Text GLabel 10550 4550 0    60   Input ~ 0
@@
 $EndComp
 $Comp
-L GND #PWR4
+L GND #PWR03
 U 1 1 58BA412A
 P 10600 3150
-F 0 "#PWR4" H 10600 2900 50  0001 C CNN
+F 0 "#PWR03" H 10600 2900 50  0001 C CNN
 F 1 "GND" H 10600 3000 50  0000 C CNN
 F 2 "" H 10600 3150 50  0000 C CNN
@@
 $EndComp
 $Comp
-L +3.3V #PWR3
+L +3.3V #PWR04
 U 1 1 58BA41CE
 P 10600 3050
-F 0 "#PWR3" H 10600 2900 50  0001 C CNN
+F 0 "#PWR04" H 10600 2900 50  0001 C CNN
 F 1 "+3.3V" H 10600 3190 50  0000 C CNN
 F 2 "" H 10600 3050 50  0000 C CNN
@@
 $EndComp
 $Comp
-L GND #PWR5
+L GND #PWR05
 U 1 1 58BABD17
 P 5450 5050
-F 0 "#PWR5" H 5450 4800 50  0001 C CNN
+F 0 "#PWR05" H 5450 4800 50  0001 C CNN
 F 1 "GND" H 5450 4900 50  0000 C CNN
 F 2 "" H 5450 5050 50  0000 C CNN
@@
 $EndComp
 $Comp
-L GND #PWR6
+L GND #PWR06
 U 1 1 58BACEDF
 P 6100 5050
-F 0 "#PWR6" H 6100 4800 50  0001 C CNN
+F 0 "#PWR06" H 6100 4800 50  0001 C CNN
 F 1 "GND" H 6100 4900 50  0000 C CNN
 F 2 "" H 6100 5050 50  0000 C CNN
@@
 $EndComp
 $Comp
-L GND #PWR8
+L GND #PWR07
 U 1 1 58BAD6B9
 P 7500 5050
-F 0 "#PWR8" H 7500 4800 50  0001 C CNN
+F 0 "#PWR07" H 7500 4800 50  0001 C CNN
 F 1 "GND" H 7500 4900 50  0000 C CNN
 F 2 "" H 7500 5050 50  0000 C CNN
@@
 $EndComp
 $Comp
-L GND #PWR7
+L GND #PWR08
 U 1 1 58BAEE31
 P 6750 5050
-F 0 "#PWR7" H 6750 4800 50  0001 C CNN
+F 0 "#PWR08" H 6750 4800 50  0001 C CNN
 F 1 "GND" H 6750 4900 50  0000 C CNN
 F 2 "" H 6750 5050 50  0000 C CNN
@@
 $EndComp
 $Comp
-L GND #PWR10
+L GND #PWR09
 U 1 1 58BAEE3D
 P 8650 5050
-F 0 "#PWR10" H 8650 4800 50  0001 C CNN
+F 0 "#PWR09" H 8650 4800 50  0001 C CNN
 F 1 "GND" H 8650 4900 50  0000 C CNN
 F 2 "" H 8650 5050 50  0000 C CNN
@@
 $EndComp
 $Comp
-L GND #PWR9
+L GND #PWR010
 U 1 1 58BAEE49
 P 8100 5050
-F 0 "#PWR9" H 8100 4800 50  0001 C CNN
+F 0 "#PWR010" H 8100 4800 50  0001 C CNN
 F 1 "GND" H 8100 4900 50  0000 C CNN
 F 2 "" H 8100 5050 50  0000 C CNN
@@
 $EndComp
 $Comp
-L GND #PWR11
+L GND #PWR011
 U 1 1 58BB11B2
 P 5450 5750
-F 0 "#PWR11" H 5450 5500 50  0001 C CNN
+F 0 "#PWR011" H 5450 5500 50  0001 C CNN
 F 1 "GND" H 5450 5600 50  0000 C CNN
 F 2 "" H 5450 5750 50  0000 C CNN
@@
 $EndComp
 $Comp
-L GND #PWR12
+L GND #PWR012
 U 1 1 58BB11BE
 P 6100 5750
-F 0 "#PWR12" H 6100 5500 50  0001 C CNN
+F 0 "#PWR012" H 6100 5500 50  0001 C CNN
 F 1 "GND" H 6100 5600 50  0000 C CNN
 F 2 "" H 6100 5750 50  0000 C CNN
@@
 $EndComp
 $Comp
-L GND #PWR14
+L GND #PWR013
 U 1 1 58BB11CA
 P 7500 5750
-F 0 "#PWR14" H 7500 5500 50  0001 C CNN
+F 0 "#PWR013" H 7500 5500 50  0001 C CNN
 F 1 "GND" H 7500 5600 50  0000 C CNN
 F 2 "" H 7500 5750 50  0000 C CNN
@@
 $EndComp
 $Comp
-L GND #PWR13
+L GND #PWR014
 U 1 1 58BB11D6
 P 6750 5750
-F 0 "#PWR13" H 6750 5500 50  0001 C CNN
+F 0 "#PWR014" H 6750 5500 50  0001 C CNN
 F 1 "GND" H 6750 5600 50  0000 C CNN
 F 2 "" H 6750 5750 50  0000 C CNN
@@
 $EndComp
 $Comp
-L GND #PWR16
+L GND #PWR015
 U 1 1 58BB11E2
 P 8650 5750
-F 0 "#PWR16" H 8650 5500 50  0001 C CNN
+F 0 "#PWR015" H 8650 5500 50  0001 C CNN
 F 1 "GND" H 8650 5600 50  0000 C CNN
 F 2 "" H 8650 5750 50  0000 C CNN
@@
 $EndComp
 $Comp
-L GND #PWR15
+L GND #PWR016
 U 1 1 58BB11EE
 P 8100 5750
-F 0 "#PWR15" H 8100 5500 50  0001 C CNN
+F 0 "#PWR016" H 8100 5500 50  0001 C CNN
 F 1 "GND" H 8100 5600 50  0000 C CNN
 F 2 "" H 8100 5750 50  0000 C CNN
