File: test_pcb/test_pcb.sch (KiCad schematic (older format))
At the start: 87 parts, among them K0 KEYSW, K1 KEYSW, K10 KEYSW, K12 KEYSW, K13 KEYSW, K14 KEYSW, K15 KEYSW, K16 KEYSW, K17 KEYSW, K18 KEYSW, K2 KEYSW, K20 KEYSW, K21 KEYSW, K22 KEYSW, K3 KEYSW, K4 KEYSW, K5 KEYSW, K6 KEYSW, K7 KEYSW, K8 KEYSW, K9 KEYSW, P1 CONN_01X10, P10 CONN_01X01, P11 CONN_01X01, P12 CONN_01X01, P13 CONN_01X01, P14 CONN_01X01, P15 CONN_01X01, P2 CONN_01X08, P3 CONN_01X06, P4 CONN_01X01, P5 CONN_01X01, P6 CONN_01X01, P7 CONN_01X01, P8 CONN_01X01, P9 CONN_01X01, U1 STP16CP05

Commit message: test somehow improved routing adding 5 more and 1mm on the right side of the board
Parts:
- added REXT0: R, Resistors_SMD:R_0603_HandSoldering, symbol R
- P1: value CONN_01X10 -> CONN_01X15; footprint Socket_Strips:Socket_Strip_Straight_1x10_Pitch2.54mm -> Socket_Strips:Socket_Strip_Straight_1x15_Pitch2.54mm; symbol CONN_01X10 -> CONN_01X15
Connections:
- net labels added: CLK, LE, OE, SDI, SDO
Changed lines of the file:
@@
 a3-17-2
 $Comp
-L GND #PWR01
+L GND #PWR1
 U 1 1 58A5AE89
 P 7750 2550
-F 0 "#PWR01" H 7750 2300 50  0001 C CNN
+F 0 "#PWR1" H 7750 2300 50  0001 C CNN
 F 1 "GND" H 7750 2400 50  0000 C CNN
 F 2 "" H 7750 2550 50  0000 C CNN
@@
 	0    1    1    0
 $EndComp
-Text GLabel 10600 2850 0    60   Input ~ 0
+Text GLabel 10600 2600 0    60   Input ~ 0
 a3-10-0
-Text GLabel 10600 2950 0    60   Input ~ 0
+Text GLabel 10600 2700 0    60   Input ~ 0
 a3-10-1
-Text GLabel 10600 2750 0    60   Input ~ 0
+Text GLabel 10600 2500 0    60   Input ~ 0
 a3-10-2
-Text GLabel 10600 3450 0    60   Input ~ 0
+Text GLabel 10600 3700 0    60   Input ~ 0
 a3-17-0
-Text GLabel 10600 3550 0    60   Input ~ 0
+Text GLabel 10600 3800 0    60   Input ~ 0
 a3-17-1
-Text GLabel 10600 3650 0    60   Input ~ 0
+Text GLabel 10600 3900 0    60   Input ~ 0
 a3-17-2
 $Comp
-L +3.3V #PWR02
+L +3.3V #PWR2
 U 1 1 58A3C033
 P 8900 2550
-F 0 "#PWR02" H 8900 2400 50  0001 C CNN
+F 0 "#PWR2" H 8900 2400 50  0001 C CNN
 F 1 "+3.3V" H 8900 2690 50  0000 C CNN
 F 2 "" H 8900 2550 50  0000 C CNN
@@
 $EndComp
 $Comp
-L CONN_01X10 P1
+L CONN_01X15 P1
 U 1 1 58A3B45B
 P 10800 3200
 F 0 "P1" H 10800 3650 50  0000 C CNN
-F 1 "CONN_01X10" V 10900 3200 50  0000 C CNN
-F 2 "Socket_Strips:Socket_Strip_Straight_1x10_Pitch2.54mm" H 10800 3200 50  0001 C CNN
+F 1 "CONN_01X15" V 10900 3200 50  0000 C CNN
+F 2 "Socket_Strips:Socket_Strip_Straight_1x15_Pitch2.54mm" H 10800 3200 50  0001 C CNN
 F 3 "" H 10800 3200 50  0000 C CNN
 	1    10800 3200
@@
 	1    0    0    -1
 $EndComp
-Text GLabel 10600 3250 0    60   Input ~ 0
+Text GLabel 10600 2800 0    60   Input ~ 0
 blue1
-Text GLabel 10600 3350 0    60   Input ~ 0
+Text GLabel 10600 2900 0    60   Input ~ 0
 red1
 Text GLabel 10550 1950 0    60   Input ~ 0
@@
 $EndComp
 $Comp
-L GND #PWR03
+L GND #PWR5
 U 1 1 58BA412A
-P 10600 3150
-F 0 "#PWR03" H 10600 2900 50  0001 C CNN
-F 1 "GND" H 10600 3000 50  0000 C CNN
-F 2 "" H 10600 3150 50  0000 C CNN
-F 3 "" H 10600 3150 50  0000 C CNN
-	1    10600 3150
+P 10600 3600
+F 0 "#PWR5" H 10600 3350 50  0001 C CNN
+F 1 "GND" H 10600 3450 50  0000 C CNN
+F 2 "" H 10600 3600 50  0000 C CNN
+F 3 "" H 10600 3600 50  0000 C CNN
+	1    10600 3600
 	0    1    1    0
 $EndComp
 $Comp
-L +3.3V #PWR04
+L +3.3V #PWR4
 U 1 1 58BA41CE
-P 10600 3050
-F 0 "#PWR04" H 10600 2900 50  0001 C CNN
-F 1 "+3.3V" H 10600 3190 50  0000 C CNN
-F 2 "" H 10600 3050 50  0000 C CNN
-F 3 "" H 10600 3050 50  0000 C CNN
-	1    10600 3050
+P 10600 3000
+F 0 "#PWR4" H 10600 2850 50  0001 C CNN
+F 1 "+3.3V" H 10600 3140 50  0000 C CNN
+F 2 "" H 10600 3000 50  0000 C CNN
+F 3 "" H 10600 3000 50  0000 C CNN
+	1    10600 3000
 	0    -1   -1   0
 $EndComp
@@
 $EndComp
 $Comp
-L GND #PWR05
+L GND #PWR6
 U 1 1 58BABD17
 P 5450 5050
-F 0 "#PWR05" H 5450 4800 50  0001 C CNN
+F 0 "#PWR6" H 5450 4800 50  0001 C CNN
 F 1 "GND" H 5450 4900 50  0000 C CNN
 F 2 "" H 5450 5050 50  0000 C CNN
@@
 $EndComp
 $Comp
-L GND #PWR06
+L GND #PWR7
 U 1 1 58BACEDF
 P 6100 5050
-F 0 "#PWR06" H 6100 4800 50  0001 C CNN
+F 0 "#PWR7" H 6100 4800 50  0001 C CNN
 F 1 "GND" H 6100 4900 50  0000 C CNN
 F 2 "" H 6100 5050 50  0000 C CNN
@@
 $EndComp
 $Comp
-L GND #PWR07
+L GND #PWR9
 U 1 1 58BAD6B9
 P 7500 5050
-F 0 "#PWR07" H 7500 4800 50  0001 C CNN
+F 0 "#PWR9" H 7500 4800 50  0001 C CNN
 F 1 "GND" H 7500 4900 50  0000 C CNN
 F 2 "" H 7500 5050 50  0000 C CNN
@@
 $EndComp
 $Comp
-L GND #PWR08
+L GND #PWR8
 U 1 1 58BAEE31
 P 6750 5050
-F 0 "#PWR08" H 6750 4800 50  0001 C CNN
+F 0 "#PWR8" H 6750 4800 50  0001 C CNN
 F 1 "GND" H 6750 4900 50  0000 C CNN
 F 2 "" H 6750 5050 50  0000 C CNN
@@
 $EndComp
 $Comp
-L GND #PWR09
+L GND #PWR11
 U 1 1 58BAEE3D
 P 8650 5050
-F 0 "#PWR09" H 8650 4800 50  0001 C CNN
+F 0 "#PWR11" H 8650 4800 50  0001 C CNN
 F 1 "GND" H 8650 4900 50  0000 C CNN
 F 2 "" H 8650 5050 50  0000 C CNN
@@
 $EndComp
 $Comp
-L GND #PWR010
+L GND #PWR10
 U 1 1 58BAEE49
 P 8100 5050
-F 0 "#PWR010" H 8100 4800 50  0001 C CNN
+F 0 "#PWR10" H 8100 4800 50  0001 C CNN
 F 1 "GND" H 8100 4900 50  0000 C CNN
 F 2 "" H 8100 5050 50  0000 C CNN
@@
 $EndComp
 $Comp
-L GND #PWR011
+L GND #PWR12
 U 1 1 58BB11B2
 P 5450 5750
-F 0 "#PWR011" H 5450 5500 50  0001 C CNN
+F 0 "#PWR12" H 5450 5500 50  0001 C CNN
 F 1 "GND" H 5450 5600 50  0000 C CNN
 F 2 "" H 5450 5750 50  0000 C CNN
@@
 $EndComp
 $Comp
-L GND #PWR012
+L GND #PWR13
 U 1 1 58BB11BE
 P 6100 5750
-F 0 "#PWR012" H 6100 5500 50  0001 C CNN
+F 0 "#PWR13" H 6100 5500 50  0001 C CNN
 F 1 "GND" H 6100 5600 50  0000 C CNN
 F 2 "" H 6100 5750 50  0000 C CNN
@@
 $EndComp
 $Comp
-L GND #PWR013
+L GND #PWR15
 U 1 1 58BB11CA
 P 7500 5750
-F 0 "#PWR013" H 7500 5500 50  0001 C CNN
+F 0 "#PWR15" H 7500 5500 50  0001 C CNN
 F 1 "GND" H 7500 5600 50  0000 C CNN
 F 2 "" H 7500 5750 50  0000 C CNN
@@
 $EndComp
 $Comp
-L GND #PWR014
+L GND #PWR14
 U 1 1 58BB11D6
 P 6750 5750
-F 0 "#PWR014" H 6750 5500 50  0001 C CNN
+F 0 "#PWR14" H 6750 5500 50  0001 C CNN
 F 1 "GND" H 6750 5600 50  0000 C CNN
 F 2 "" H 6750 5750 50  0000 C CNN
@@
 $EndComp
 $Comp
-L GND #PWR015
+L GND #PWR17
 U 1 1 58BB11E2
 P 8650 5750
-F 0 "#PWR015" H 8650 5500 50  0001 C CNN
+F 0 "#PWR17" H 8650 5500 50  0001 C CNN
 F 1 "GND" H 8650 5600 50  0000 C CNN
 F 2 "" H 8650 5750 50  0000 C CNN
@@
 $EndComp
 $Comp
-L GND #PWR016
+L GND #PWR16
 U 1 1 58BB11EE
 P 8100 5750
-F 0 "#PWR016" H 8100 5500 50  0001 C CNN
+F 0 "#PWR16" H 8100 5500 50  0001 C CNN
 F 1 "GND" H 8100 5600 50  0000 C CNN
 F 2 "" H 8100 5750 50  0000 C CNN
@@
 	0    -1   1    0
 $EndComp
+Text GLabel 10600 3500 0    60   Input ~ 0
+SDI
+Text GLabel 10600 3400 0    60   Input ~ 0
+CLK
+Text GLabel 10600 3300 0    60   Input ~ 0
+LE
+Text GLabel 10600 3100 0    60   Input ~ 0
+SDO
+Text GLabel 10600 3200 0    60   Input ~ 0
+OE
+Text GLabel 8900 2750 2    60   Input ~ 0
+SDO
+Text GLabel 8900 2850 2    60   Input ~ 0
+OE
+Text GLabel 7750 2850 0    60   Input ~ 0
+LE
+Text GLabel 7750 2750 0    60   Input ~ 0
+CLK
+Text GLabel 7750 2650 0    60   Input ~ 0
+SDI
+$Comp
+L R REXT0
+U 1 1 58BB9157
+P 9150 2650
+F 0 "REXT0" V 9230 2650 50  0000 C CNN
+F 1 "R" V 9150 2650 50  0000 C CNN
+F 2 "Resistors_SMD:R_0603_HandSoldering" H 9150 2650 60  0001 C CNN
+F 3 "" H 9150 2650 60  0000 C CNN
+	1    9150 2650
+	0    1    -1   0
+$EndComp
+$Comp
+L GND #PWR3
+U 1 1 58BB9A32
+P 9400 2650
+F 0 "#PWR3" H 9400 2400 50  0001 C CNN
+F 1 "GND" H 9400 2500 50  0000 C CNN
+F 2 "" H 9400 2650 50  0000 C CNN
+F 3 "" H 9400 2650 50  0000 C CNN
+	1    9400 2650
+	0    -1   -1   0
+$EndComp
 $EndSCHEMATC

Commit message: test groundplanes
Parts:
- JP4: footprint Pin_Headers:Pin_Header_Angled_1x02_Pitch1.27mm -> cherry_rgb:Pin_Header_Angled_1x02_Pitch1.27mm_flipped
