File: tp_pcb/tp_pcb.kicad_pcb (KiCad board)
At the start: 2 copper layers, 66.5 x 76 mm, 34 parts, among them K0 KEYSW, K1 KEYSW, K2 KEYSW, K3 KEYSW, K4 KEYSW, K5 KEYSW, K6 KEYSW, P0 CONN_01X08, P1 CONN_01X08, P2 CONN_01X06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

Commit message: tp silkscreen touchup and a few final tweaks
Parts:
- LVC9_HOLES: footprint cherry_rgb:LVC9_HOLES -> cherry_rgb:LVC9_HOLES_for_tptest
Other:
- board text added: "2 1 0 C D V R G"
- board text added: "G R V D C"
- board text added: "a0 a1 a2 a3 c0 r0 r1 c1"
- board text added: "b0 g0 red0 b1 red1 g1"
Changed lines of the file:
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@@
     (links 59)
     (no_connects 0)
-    (area 105.674999 33.424999 172.325001 109.575001)
+    (area 90.325799 33.325799 185.674201 111.3176)
     (thickness 1.6)
-    (drawings 10)
-    (tracks 337)
+    (drawings 14)
+    (tracks 336)
     (zones 0)
     (modules 34)
@@
     (add_net red1)
   )
-  (module cherry_rgb:LVC9_HOLES (layer F.Cu)
-    (at 138 51.5)
-    (fp_text reference LVC9_HOLES (at 0 -5.25) (layer F.SilkS)
-      (effects (font (size 1 1) (thickness 0.15)))
-    )
-    (fp_text value "LVC9 Attach" (at 0 5.5) (layer F.Fab)
-      (effects (font (size 1 1) (thickness 0.15)))
-    )
-    (fp_arc (start -14.5 21) (end -14.5 22.5) (angle 90) (layer B.SilkS) (width 0.15))
-    (fp_arc (start 12 21) (end 13.5 21) (angle 90) (layer B.SilkS) (width 0.15))
-    (fp_arc (start 12 -6) (end 12 -7.5) (angle 90) (layer B.SilkS) (width 0.15))
-    (fp_arc (start -14.5 -6) (end -16 -6) (angle 90) (layer B.SilkS) (width 0.15))
-    (fp_line (start -14.5 -7.5) (end 12 -7.5) (layer B.SilkS) (width 0.15))
-    (fp_line (start 13.5 -6) (end 13.5 21) (layer B.SilkS) (width 0.15))
-    (fp_line (start 12 22.5) (end -14.5 22.5) (layer B.SilkS) (width 0.15))
-    (fp_line (start -16 21) (end -16 -6) (layer B.SilkS) (width 0.15))
-    (pad "" np_thru_hole circle (at -8.5 8) (size 2.5 2.5) (drill 2.5) (layers *.Cu *.Mask))
-    (pad "" np_thru_hole circle (at 8.5 8) (size 2.5 2.5) (drill 2.5) (layers *.Cu *.Mask))
-    (pad "" np_thru_hole circle (at 9.5 0) (size 2.5 2.5) (drill 2.5) (layers *.Cu *.Mask))
-    (pad "" np_thru_hole circle (at 0 0) (size 8 8) (drill 8) (layers *.Cu *.Mask))
-    (pad "" np_thru_hole circle (at -9.5 0) (size 2.5 2.5) (drill 2.5) (layers *.Cu *.Mask))
-  )
   (module cherry_rgb:tgbugs_sig (layer B.Cu)
     (at 152 99.25 180)
@@
     (tags "connector molex picoblade smt")
     (attr smd)
-    (fp_text reference P0 (at 0 3.5) (layer B.SilkS)
+    (fp_text reference P0 (at 0 -1) (layer B.SilkS)
       (effects (font (size 1 1) (thickness 0.15)) (justify mirror))
     )
@@
     (descr "Through hole straight socket strip, 1x08, 2.54mm pitch, single row")
     (tags "Through hole socket strip THT 1x08 2.54mm single row")
-    (fp_text reference P1 (at 0 -2.33) (layer F.SilkS)
+    (fp_text reference P1 (at 2.5 20) (layer F.SilkS)
       (effects (font (size 1 1) (thickness 0.15)))
     )
@@
     (pad HOLE np_thru_hole circle (at 0 0) (size 3.9878 3.9878) (drill 3.9878) (layers *.Cu))
   )
+  (module cherry_rgb:LVC9_HOLES_for_tptest (layer F.Cu)
+    (at 138 51.5)
+    (fp_text reference LVC9_HOLES (at 0 -5.25) (layer F.SilkS)
+      (effects (font (size 1 1) (thickness 0.15)))
+    )
+    (fp_text value "LVC9 Attach" (at 0 5.5) (layer F.Fab)
+      (effects (font (size 1 1) (thickness 0.15)))
+    )
+    (fp_arc (start -14.5 21) (end -14.5 22.5) (angle 90) (layer B.SilkS) (width 0.15))
+    (fp_arc (start 12 21) (end 13.5 21) (angle 90) (layer B.SilkS) (width 0.15))
+    (fp_arc (start 12 -6) (end 12 -7.5) (angle 90) (layer B.SilkS) (width 0.15))
+    (fp_arc (start -14.5 -6) (end -16 -6) (angle 90) (layer B.SilkS) (width 0.15))
+    (fp_line (start -14.5 -7.5) (end 12 -7.5) (layer B.SilkS) (width 0.15))
+    (fp_line (start 13.5 -6) (end 13.5 21) (layer B.SilkS) (width 0.15))
+    (fp_line (start 12 22.5) (end -14.5 22.5) (layer B.SilkS) (width 0.15))
+    (pad "" np_thru_hole circle (at -8.5 8) (size 2.5 2.5) (drill 2.5) (layers *.Cu *.Mask))
+    (pad "" np_thru_hole circle (at 8.5 8) (size 2.5 2.5) (drill 2.5) (layers *.Cu *.Mask))
+    (pad "" np_thru_hole circle (at 9.5 0) (size 2.5 2.5) (drill 2.5) (layers *.Cu *.Mask))
+    (pad "" np_thru_hole circle (at 0 0) (size 8 8) (drill 8) (layers *.Cu *.Mask))
+    (pad "" np_thru_hole circle (at -9.5 0) (size 2.5 2.5) (drill 2.5) (layers *.Cu *.Mask))
+  )
+  (gr_text "b0\ng0\nred0\nb1\nred1\ng1" (at 125.25 63.25) (layer F.SilkS)
+    (effects (font (size 1.5 1.5) (thickness 0.3)))
+  )
+  (gr_text "a0\na1\na2\na3\nc0\nr0\nr1\nc1" (at 111 82) (layer F.SilkS)
+    (effects (font (size 1.5 1.5) (thickness 0.3)))
+  )
+  (gr_text "G\nR\nV\nD\nC" (at 152 83.75) (layer F.SilkS)
+    (effects (font (size 1.5 1.5) (thickness 0.3)))
+  )
+  (gr_text "2 1 0 C D V R G" (at 124.25 95.5) (layer B.SilkS)
+    (effects (font (size 0.7 0.7) (thickness 0.1)) (justify mirror))
+  )
   (gr_line (start 157 89.5) (end 157 33.5) (angle 90) (layer Edge.Cuts) (width 0.15))
   (gr_line (start 172.25 90.5) (end 158 90.5) (angle 90) (layer Edge.Cuts) (width 0.15))
@@
   (segment (start 106.0854 73.0021) (end 106.0854 84.0354) (width 0.25) (layer B.Cu) (net 5))
   (segment (start 150.04 37.92) (end 131.04 37.92) (width 0.25) (layer B.Cu) (net 5))
+  (segment (start 108 88.49) (end 108.849999 87.640001) (width 0.25) (layer B.Cu) (net 6))
+  (segment (start 108.849999 87.640001) (end 119.109999 87.640001) (width 0.25) (layer B.Cu) (net 6))
+  (segment (start 119.109999 87.640001) (end 124.5 82.25) (width 0.25) (layer B.Cu) (net 6))
+  (segment (start 124.5 82.25) (end 128.5 82.25) (width 0.25) (layer B.Cu) (net 6))
+  (segment (start 133.340947 76.5) (end 138.343554 76.5) (width 0.25) (layer B.Cu) (net 6))
+  (segment (start 128.5 82.25) (end 130.840947 79.909053) (width 0.25) (layer B.Cu) (net 6))
+  (segment (start 130.840947 79.909053) (end 130.840947 79) (width 0.25) (layer B.Cu) (net 6))
+  (segment (start 130.840947 79) (end 133.340947 76.5) (width 0.25) (layer B.Cu) (net 6))
+  (segment (start 138.343554 76.5) (end 138.923554 75.92) (width 0.25) (layer B.Cu) (net 6))
+  (segment (start 138.923554 75.92) (end 140.54 75.92) (width 0.25) (layer B.Cu) (net 6))
   (segment (start 143 60.75) (end 143 59.38) (width 0.25) (layer B.Cu) (net 6))
   (segment (start 143 59.38) (end 140.54 56.92) (width 0.25) (layer B.Cu) (net 6))
@@
   (segment (start 141.9879 61.75) (end 141.9879 74.4721) (width 0.25) (layer B.Cu) (net 6))
   (segment (start 141.9879 61.75) (end 142 61.75) (width 0.25) (layer B.Cu) (net 6))
-  (segment (start 108 88.49) (end 108.599999 87.890001) (width 0.25) (layer B.Cu) (net 6) (status 10))
-  (segment (start 108.599999 87.890001) (end 118.859999 87.890001) (width 0.25) (layer B.Cu) (net 6))
-  (segment (start 118.859999 87.890001) (end 124.5 82.25) (width 0.25) (layer B.Cu) (net 6))
-  (segment (start 124.5 82.25) (end 128.5 82.25) (width 0.25) (layer B.Cu) (net 6))
-  (segment (start 133.340947 76.5) (end 138.343554 76.5) (width 0.25) (layer B.Cu) (net 6))
-  (segment (start 138.923554 75.92) (end 140.54 75.92) (width 0.25) (layer B.Cu) (net 6))
-  (segment (start 128.5 82.25) (end 130.840947 79.909053) (width 0.25) (layer B.Cu) (net 6))
-  (segment (start 130.840947 79.909053) (end 130.840947 79) (width 0.25) (layer B.Cu) (net 6))
-  (segment (start 130.840947 79) (end 133.340947 76.5) (width 0.25) (layer B.Cu) (net 6))
-  (segment (start 138.343554 76.5) (end 138.923554 75.92) (width 0.25) (layer B.Cu) (net 6))
   (segment (start 141.9879 74.4721) (end 140.54 75.92) (width 0.25) (layer B.Cu) (net 6))
   (segment (start 125.8303 94.92) (end 126.125 94.6253) (width 0.25) (layer B.Cu) (net 7))
@@
   (segment (start 131.35 57) (end 131.35 57.7861) (width 0.25) (layer B.Cu) (net 25))
   (segment (start 131.35 57.7861) (end 131.35 62) (width 0.25) (layer B.Cu) (net 25))
-  (segment (start 113.6447 91.03) (end 108 91.03) (width 0.25) (layer B.Cu) (net 26))
-  (segment (start 116.1747 88.5) (end 114 90.6747) (width 0.25) (layer B.Cu) (net 26))
-  (segment (start 114 90.6747) (end 113.6447 91.03) (width 0.25) (layer B.Cu) (net 26))
+  (segment (start 115 88.25) (end 112.22 91.03) (width 0.25) (layer B.Cu) (net 26))
+  (segment (start 112.22 91.03) (end 108 91.03) (width 0.25) (layer B.Cu) (net 26))
+  (segment (start 119.25 88.25) (end 115 88.25) (width 0.25) (layer B.Cu) (net 26))
+  (segment (start 124.75 82.75) (end 119.25 88.25) (width 0.25) (layer B.Cu) (net 26))
   (segment (start 143.5 61) (end 143.5 59.045) (width 0.25) (layer B.Cu) (net 26))
   (segment (start 143.5 59.045) (end 142.455 58) (width 0.25) (layer B.Cu) (net 26))
@@
   (segment (start 130.65 81) (end 128.9 82.75) (width 0.25) (layer B.Cu) (net 26))
   (segment (start 128.9 82.75) (end 124.75 82.75) (width 0.25) (layer B.Cu) (net 26))
-  (segment (start 124.75 82.75) (end 119 88.5) (width 0.25) (layer B.Cu) (net 26))
-  (segment (start 119 88.5) (end 116.1747 88.5) (width 0.25) (layer B.Cu) (net 26))
   (segment (start 131.35 81) (end 131.35 79.127358) (width 0.25) (layer B.Cu) (net 26))
   (segment (start 141.191399 77.388001) (end 142.455 76.1244) (width 0.25) (layer B.Cu) (net 26))
@@
       )
     )
+  )
+  (zone (net 0) (net_name "") (layer B.Cu) (hatch edge 0.508)
+    (connect_pads (clearance 0.25))
+    (min_thickness 0.254)
+    (keepout (tracks allowed) (vias allowed) (copperpour not_allowed))
+    (fill yes (arc_segments 16) (thermal_gap 0.508) (thermal_bridge_width 0.508))
+    (polygon
+      (pts
+        (xy 130 88.75) (xy 129.75 89) (xy 129.25 88.5) (xy 129.5 88.25)
+      )
+    )
